File: flm-wagenbeleuchtung.kicad_sch (KiCad schematic)
At the start: 27 parts

Commit message: v2
Parts:
- added C5, C6: 200u, Capacitor_Tantalum_SMD:CP_EIA-7343-31_Kemet-D_Pad2.25x2.55mm_HandSolder, symbol Device:C_Polarized
Connections:
- net GND: now also C5.2, C6.2; no longer RV1.3
- net VCC: now also C5.1, C6.1
- no-connect marks 3 -> 4
Changed lines of the file:
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@@
   (junction (at 77.47 73.66) (diameter 0) (color 0 0 0 0)
   )
+  (junction (at 172.72 59.69) (diameter 0) (color 0 0 0 0)
+  )
   (junction (at 135.89 52.07) (diameter 0) (color 0 0 0 0)
   )
@@
   (junction (at 119.38 73.66) (diameter 0) (color 0 0 0 0)
   )
+  (junction (at 153.67 52.07) (diameter 0) (color 0 0 0 0)
+  )
   (junction (at 135.89 59.69) (diameter 0) (color 0 0 0 0)
   )
@@
   (junction (at 119.38 104.14) (diameter 0) (color 0 0 0 0)
   )
+  (junction (at 153.67 59.69) (diameter 0) (color 0 0 0 0)
+  )
   (junction (at 100.33 52.07) (diameter 0) (color 0 0 0 0)
   )
@@
   )
   (junction (at 77.47 104.14) (diameter 0) (color 0 0 0 0)
+  )
+  (junction (at 172.72 52.07) (diameter 0) (color 0 0 0 0)
   )
   (junction (at 100.33 59.69) (diameter 0) (color 0 0 0 0)
@@
   (no_connect (at 25.4 57.15))
   (no_connect (at 25.4 36.83))
+  (no_connect (at 77.47 55.88))
   (wire (pts (xy 25.4 57.15) (xy 50.8 57.15))
     (stroke (width 0) (type default) (color 0 0 0 0))
@@
     (stroke (width 0) (type default) (color 0 0 0 0))
   )
+  (wire (pts (xy 153.67 59.69) (xy 172.72 59.69))
+    (stroke (width 0) (type default) (color 0 0 0 0))
+  )
   (wire (pts (xy 119.38 66.04) (xy 119.38 73.66))
     (stroke (width 0) (type default) (color 0 0 0 0))
@@
     (stroke (width 0) (type default) (color 0 0 0 0))
   )
-  (wire (pts (xy 77.47 55.88) (xy 77.47 59.69))
-    (stroke (width 0) (type default) (color 0 0 0 0))
-  )
   (wire (pts (xy 119.38 83.82) (xy 116.84 83.82))
     (stroke (width 0) (type default) (color 0 0 0 0))
@@
     (stroke (width 0) (type default) (color 0 0 0 0))
   )
+  (wire (pts (xy 172.72 59.69) (xy 191.77 59.69))
+    (stroke (width 0) (type default) (color 0 0 0 0))
+  )
   (wire (pts (xy 119.38 93.98) (xy 119.38 104.14))
     (stroke (width 0) (type default) (color 0 0 0 0))
@@
     (stroke (width 0) (type default) (color 0 0 0 0))
   )
+  (wire (pts (xy 172.72 52.07) (xy 191.77 52.07))
+    (stroke (width 0) (type default) (color 0 0 0 0))
+  )
   (wire (pts (xy 86.36 83.82) (xy 77.47 83.82))
     (stroke (width 0) (type default) (color 0 0 0 0))
@@
   )
   (wire (pts (xy 86.36 93.98) (xy 77.47 93.98))
+    (stroke (width 0) (type default) (color 0 0 0 0))
+  )
+  (wire (pts (xy 153.67 52.07) (xy 172.72 52.07))
     (stroke (width 0) (type default) (color 0 0 0 0))
   )
@@
     )
     (property "Datasheet" "~" (id 3) (at 153.67 55.88 0)
+      (effects (font (size 1.27 1.27)) hide)
+    )
+    (pin "1")
+    (pin "2")
+  )
+  (symbol (lib_id "Device:C_Polarized") (at 172.72 55.88 0) (unit 1)
+    (in_bom yes) (on_board yes) (fields_autoplaced)
+    (property "Reference" "C5" (id 0) (at 175.641 54.1563 0)
+      (effects (font (size 1.27 1.27)) (justify left))
+    )
+    (property "Value" "200u" (id 1) (at 175.641 56.6932 0)
+      (effects (font (size 1.27 1.27)) (justify left))
+    )
+    (property "Footprint" "Capacitor_Tantalum_SMD:CP_EIA-7343-31_Kemet-D_Pad2.25x2.55mm_HandSolder" (id 2) (at 173.6852 59.69 0)
+      (effects (font (size 1.27 1.27)) hide)
+    )
+    (property "Datasheet" "~" (id 3) (at 172.72 55.88 0)
       (effects (font (size 1.27 1.27)) hide)
     )
@@
     (pin "2")
   )
+  (symbol (lib_id "Device:C_Polarized") (at 191.77 55.88 0) (unit 1)
+    (in_bom yes) (on_board yes) (fields_autoplaced)
+    (property "Reference" "C6" (id 0) (at 194.691 54.1563 0)
+      (effects (font (size 1.27 1.27)) (justify left))
+    )
+    (property "Value" "200u" (id 1) (at 194.691 56.6932 0)
+      (effects (font (size 1.27 1.27)) (justify left))
+    )
+    (property "Footprint" "Capacitor_Tantalum_SMD:CP_EIA-7343-31_Kemet-D_Pad2.25x2.55mm_HandSolder" (id 2) (at 192.7352 59.69 0)
+      (effects (font (size 1.27 1.27)) hide)
+    )
+    (property "Datasheet" "~" (id 3) (at 191.77 55.88 0)
+      (effects (font (size 1.27 1.27)) hide)
+    )
+    (pin "1")
+    (pin "2")
+  )
   (symbol (lib_id "Device:C_Polarized") (at 135.89 55.88 0) (unit 1)
     (in_bom yes) (on_board yes) (fields_autoplaced)
@@
       (reference "C4") (unit 1) (value "200u") (footprint "Capacitor_Tantalum_SMD:CP_EIA-7343-31_Kemet-D_Pad2.25x2.55mm_HandSolder")
     )
+    (path "/034f9fb7-343a-4f1e-97dc-028c15eef090"
+      (reference "C5") (unit 1) (value "200u") (footprint "Capacitor_Tantalum_SMD:CP_EIA-7343-31_Kemet-D_Pad2.25x2.55mm_HandSolder")
+    )
+    (path "/e8f81917-814d-47c5-9e15-0781fa689d6b"
+      (reference "C6") (unit 1) (value "200u") (footprint "Capacitor_Tantalum_SMD:CP_EIA-7343-31_Kemet-D_Pad2.25x2.55mm_HandSolder")
+    )
     (path "/cf49d850-1e17-4d42-9f03-5ca89dd17838"
