File: flm-wagenbeleuchtung/flm-wagenbeleuchtung.kicad_sch (KiCad schematic)
At the start: 29 parts

Commit message: flm: 3k3
Parts:
- R1, R2, R3, R4, R5: value 120 -> 3K3
- R6: value R -> 10K
Changed lines of the file:
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@@
     (in_bom yes) (on_board yes) (fields_autoplaced)
     (property "Reference" "R5" (id 0) (at 113.03 109.5842 90))
-    (property "Value" "120" (id 1) (at 113.03 112.1211 90))
+    (property "Value" "3K3" (id 1) (at 113.03 112.1211 90))
     (property "Footprint" "Resistor_SMD:R_1206_3216Metric_Pad1.30x1.75mm_HandSolder" (id 2) (at 113.03 116.078 90)
       (effects (font (size 1.27 1.27)) hide)
@@
     (in_bom yes) (on_board yes) (fields_autoplaced)
     (property "Reference" "R2" (id 0) (at 113.03 79.1042 90))
-    (property "Value" "120" (id 1) (at 113.03 81.6411 90))
+    (property "Value" "3K3" (id 1) (at 113.03 81.6411 90))
     (property "Footprint" "Resistor_SMD:R_1206_3216Metric_Pad1.30x1.75mm_HandSolder" (id 2) (at 113.03 85.598 90)
       (effects (font (size 1.27 1.27)) hide)
@@
     (in_bom yes) (on_board yes) (fields_autoplaced)
     (property "Reference" "R1" (id 0) (at 113.03 68.9442 90))
-    (property "Value" "120" (id 1) (at 113.03 71.4811 90))
+    (property "Value" "3K3" (id 1) (at 113.03 71.4811 90))
     (property "Footprint" "Resistor_SMD:R_1206_3216Metric_Pad1.30x1.75mm_HandSolder" (id 2) (at 113.03 75.438 90)
       (effects (font (size 1.27 1.27)) hide)
@@
     (in_bom yes) (on_board yes) (fields_autoplaced)
     (property "Reference" "R3" (id 0) (at 113.03 89.2642 90))
-    (property "Value" "120" (id 1) (at 113.03 91.8011 90))
+    (property "Value" "3K3" (id 1) (at 113.03 91.8011 90))
     (property "Footprint" "Resistor_SMD:R_1206_3216Metric_Pad1.30x1.75mm_HandSolder" (id 2) (at 113.03 95.758 90)
       (effects (font (size 1.27 1.27)) hide)
@@
     (in_bom yes) (on_board yes) (fields_autoplaced)
     (property "Reference" "R4" (id 0) (at 113.03 99.4242 90))
-    (property "Value" "120" (id 1) (at 113.03 101.9611 90))
+    (property "Value" "3K3" (id 1) (at 113.03 101.9611 90))
     (property "Footprint" "Resistor_SMD:R_1206_3216Metric_Pad1.30x1.75mm_HandSolder" (id 2) (at 113.03 105.918 90)
       (effects (font (size 1.27 1.27)) hide)
@@
     (in_bom yes) (on_board yes) (fields_autoplaced)
     (property "Reference" "R6" (id 0) (at 97.79 119.7442 90))
-    (property "Value" "R" (id 1) (at 97.79 122.2811 90))
+    (property "Value" "10K" (id 1) (at 97.79 122.2811 90))
     (property "Footprint" "Resistor_SMD:R_1206_3216Metric_Pad1.30x1.75mm_HandSolder" (id 2) (at 97.79 122.682 90)
       (effects (font (size 1.27 1.27)) hide)
@@
     )
     (path "/b1d535f1-db1b-4494-9e30-3b9a4bed4d52"
-      (reference "R1") (unit 1) (value "120") (footprint "Resistor_SMD:R_1206_3216Metric_Pad1.30x1.75mm_HandSolder")
+      (reference "R1") (unit 1) (value "3K3") (footprint "Resistor_SMD:R_1206_3216Metric_Pad1.30x1.75mm_HandSolder")
     )
     (path "/46303e58-1547-4130-86b5-f2bda87c84a8"
-      (reference "R2") (unit 1) (value "120") (footprint "Resistor_SMD:R_1206_3216Metric_Pad1.30x1.75mm_HandSolder")
+      (reference "R2") (unit 1) (value "3K3") (footprint "Resistor_SMD:R_1206_3216Metric_Pad1.30x1.75mm_HandSolder")
     )
     (path "/e84651d0-e334-4805-a1cb-2696e88cf6f5"
-      (reference "R3") (unit 1) (value "120") (footprint "Resistor_SMD:R_1206_3216Metric_Pad1.30x1.75mm_HandSolder")
+      (reference "R3") (unit 1) (value "3K3") (footprint "Resistor_SMD:R_1206_3216Metric_Pad1.30x1.75mm_HandSolder")
     )
     (path "/ea64b4ed-9c67-4795-ba77-b5eae9daeb64"
-      (reference "R4") (unit 1) (value "120") (footprint "Resistor_SMD:R_1206_3216Metric_Pad1.30x1.75mm_HandSolder")
+      (reference "R4") (unit 1) (value "3K3") (footprint "Resistor_SMD:R_1206_3216Metric_Pad1.30x1.75mm_HandSolder")
     )
     (path "/3221ac2b-cb74-4dd4-9657-801da79bca99"
-      (reference "R5") (unit 1) (value "120") (footprint "Resistor_SMD:R_1206_3216Metric_Pad1.30x1.75mm_HandSolder")
+      (reference "R5") (unit 1) (value "3K3") (footprint "Resistor_SMD:R_1206_3216Metric_Pad1.30x1.75mm_HandSolder")
     )
     (path "/f11b3517-e24d-463c-aa0a-6cdb386f637e"
-      (reference "R6") (unit 1) (value "R") (footprint "Resistor_SMD:R_1206_3216Metric_Pad1.30x1.75mm_HandSolder")
+      (reference "R6") (unit 1) (value "10K") (footprint "Resistor_SMD:R_1206_3216Metric_Pad1.30x1.75mm_HandSolder")
     )
     (path "/a0cc0dd8-596a-43aa-86b8-bc157c22a5e9"
