File: minitrix-wagenbeleuchtung/minitrix-wagenbeleuchtung.kicad_pcb (KiCad board)
At the start: 2 copper layers, 137 x 12 mm, 56 parts, among them J1 Conn_01x01, J10 Conn_01x01, J11 Conn_01x01, J12 Conn_01x01, J13 Conn_01x01, J14 Conn_01x01, J15 Conn_01x01, J16 Conn_01x01, J2 Conn_01x01, J20 Conn_01x01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

Commit message: minitrix v1
Parts:
- removed R6: R, Resistor_SMD:R_1206_3216Metric_Pad1.30x1.75mm_HandSolder
- removed REF** (x2): TestPoint_Pad_D4.0mm, TestPoint:TestPoint_Pad_D4.0mm
- removed SCHLUSS+, SCHLUSS-: Conn_01x01_Male, Connector_Wire:SolderWirePad_1x01_SMD_1x2mm
- J1, J2: footprint TestPoint:TestPoint_Pad_1.5x1.5mm -> Local:Minitrix_Pad; moved to B.Cu
- moved J21 63.1 mm to (180.5, 45.0), turned to 90 degrees
- moved J20 62.6 mm to (177.5, 45.0), turned to 90 degrees
- moved J1 60.8 mm to (70.0, 50.0), turned to 180 degrees
- moved J10 60.2 mm to (76.5, 45.2)
- moved J11 57.7 mm to (79.0, 45.2)
- moved J2 57.2 mm to (179.0, 50.0), turned to 180 degrees
- moved J12 57.1 mm to (81.5, 45.2)
- moved J13 57.0 mm to (84.0, 45.2)
- moved JP21 56.6 mm to (164.1, 45.7), turned to -90 degrees
- moved J22 54.5 mm to (179.0, 55.0), turned to 90 degrees
- moved J14 54.1 mm to (86.5, 45.2)
- moved J15 53.8 mm to (89.0, 45.2)
- moved J16 53.8 mm to (91.5, 45.2)
- moved JP20 52.0 mm to (161.1, 45.7), turned to -90 degrees
- moved R20 51.5 mm to (172.6, 45.5), turned to 180 degrees
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Connections:
- net Net-(D100-+) renamed /BRIDGE+
- net Net-(D100--) renamed /BRIDGE-
- net Net-(J20-Pin_1) renamed /LHLED
- net Net-(J21-Pin_1) renamed /LVLED
Routing:
- net GND: track 301.0 -> 130.4 mm, vias 9 -> 0
- net /AUX1: track 0.00 -> 156.6 mm, vias 0 -> 2
- net /TRACK_R: track 0.00 -> 116.8 mm
- net /TRACK_L: track 0.00 -> 110.2 mm, vias 0 -> 9
- net /LV: track 0.00 -> 104.0 mm, vias 0 -> 8
- net /TRACK_P: track 101.4 -> 0.00 mm, vias 2 -> 0
- net /LH: track 0.00 -> 90.7 mm, vias 0 -> 4
- net Net-(JP1-B): track 0.00 -> 35.2 mm, vias 0 -> 6
- net /BRIDGE-: track 0.00 -> 18.4 mm, vias 0 -> 2
- net VCC: track 176.9 -> 161.1 mm
- net /TRACK_N: track 13.5 -> 0.00 mm, vias 2 -> 0
- net /LVLED: track 0.00 -> 13.2 mm, vias 0 -> 2
- net Net-(SCHLUSS-1-Pin_1): track 5.60 -> 0.00 mm
- net /LHLED: track 0.00 -> 3.61 mm
- net Net-(D3-A): track 4.58 -> 7.89 mm, vias 0 -> 2
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Other:
- board text added: "AUX1 INNENBEL."
- board text added: "BRIDGE+|BRIDGE-|INNEN-GND|LH-GND|LV-GND"
- board text added: "GND"
- board text added: "LH GELB"
- board text added: "LH+/LV+"
- board text added: "LH-"
- board text added: "LV WEIß"
- board text added: "LV-"
- board text added: "TRACK L SCHWARZ"
- board text added: "TRACK R ROT"
- board text added: "VS+ BLAU"
