File: minitrix-wagenbeleuchtung/minitrix-wagenbeleuchtung.kicad_sch (KiCad schematic)
At the start: 51 parts, among them J1 Conn_01x01, J10 Conn_01x01, J11 Conn_01x01, J12 Conn_01x01, J13 Conn_01x01, J14 Conn_01x01, J15 Conn_01x01, J16 Conn_01x01, J2 Conn_01x01, J20 Conn_01x01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

Commit message: minitrix v1
Parts:
- J1, J2: footprint TestPoint:TestPoint_Pad_1.5x1.5mm -> Local:Minitrix_Pad
Connections:
- net LHLED: now reaches J20.1 (Pin_1), R20.1
- net LVLED: now reaches J21.1 (Pin_1), R21.1
- net BRIDGE+: now reaches D100.1 (+), RV1.1
- net BRIDGE-: now reaches D100.2 (-), JP2.2 (B)
Other:
- moved on the sheet: JP1, JP2
Changed lines of the file:
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@@
   (junction (at 30.48 100.33) (diameter 0) (color 0 0 0 0)
   )
-  (junction (at 114.3 33.02) (diameter 0) (color 0 0 0 0)
-  )
   (junction (at 160.02 146.05) (diameter 0) (color 0 0 0 0)
   )
@@
   )
   (junction (at 54.61 120.65) (diameter 0) (color 0 0 0 0)
+  )
+  (junction (at 114.3 50.8) (diameter 0) (color 0 0 0 0)
   )
   (junction (at 72.39 80.01) (diameter 0) (color 0 0 0 0)
@@
     (stroke (width 0) (type default))
   )
+  (wire (pts (xy 133.35 46.99) (xy 133.35 50.8))
+    (stroke (width 0) (type default))
+  )
+  (wire (pts (xy 166.37 46.99) (xy 166.37 58.42))
+    (stroke (width 0) (type default))
+  )
   (wire (pts (xy 157.48 36.83) (xy 157.48 50.8))
     (stroke (width 0) (type default))
@@
     (stroke (width 0) (type default))
   )
-  (wire (pts (xy 114.3 33.02) (xy 114.3 24.13))
-    (stroke (width 0) (type default))
-  )
   (wire (pts (xy 72.39 80.01) (xy 114.3 80.01))
     (stroke (width 0) (type default))
@@
     (stroke (width 0) (type default))
   )
-  (wire (pts (xy 114.3 80.01) (xy 114.3 33.02))
+  (wire (pts (xy 114.3 24.13) (xy 114.3 50.8))
     (stroke (width 0) (type default))
   )
@@
     (stroke (width 0) (type default))
   )
+  (wire (pts (xy 114.3 50.8) (xy 114.3 80.01))
+    (stroke (width 0) (type default))
+  )
   (wire (pts (xy 76.2 31.75) (xy 88.9 31.75))
     (stroke (width 0) (type default))
@@
     (stroke (width 0) (type default))
   )
-  (wire (pts (xy 186.69 33.02) (xy 179.07 33.02))
+  (wire (pts (xy 166.37 33.02) (xy 186.69 33.02))
     (stroke (width 0) (type default))
   )
@@
     (stroke (width 0) (type default))
   )
+  (wire (pts (xy 133.35 50.8) (xy 114.3 50.8))
+    (stroke (width 0) (type default))
+  )
   (wire (pts (xy 30.48 120.65) (xy 30.48 138.43))
     (stroke (width 0) (type default))
@@
     (stroke (width 0) (type default))
   )
-  (wire (pts (xy 138.43 33.02) (xy 114.3 33.02))
-    (stroke (width 0) (type default))
-  )
   (wire (pts (xy 232.41 71.12) (xy 228.6 71.12))
     (stroke (width 0) (type default))
   )
-  (wire (pts (xy 171.45 33.02) (xy 166.37 33.02))
-    (stroke (width 0) (type default))
-  )
   (wire (pts (xy 74.93 196.85) (xy 104.14 196.85))
     (stroke (width 0) (type default))
@@
     (stroke (width 0) (type default))
   )
-  (wire (pts (xy 146.05 33.02) (xy 153.67 33.02))
+  (wire (pts (xy 133.35 33.02) (xy 153.67 33.02))
     (stroke (width 0) (type default))
   )
@@
     (stroke (width 0) (type default))
   )
-  (wire (pts (xy 166.37 33.02) (xy 166.37 58.42))
+  (wire (pts (xy 166.37 33.02) (xy 166.37 39.37))
     (stroke (width 0) (type default))
   )
@@
     (stroke (width 0) (type default))
   )
+  (wire (pts (xy 133.35 33.02) (xy 133.35 39.37))
+    (stroke (width 0) (type default))
+  )
   (wire (pts (xy 194.31 25.4) (xy 194.31 21.59))
     (stroke (width 0) (type default))
@@
     (effects (font (size 1.27 1.27)) (justify left bottom))
   )
+  (label "BRIDGE-" (at 175.26 33.02 0) (fields_autoplaced)
+    (effects (font (size 1.27 1.27)) (justify left bottom))
+  )
+  (label "LVLED" (at 180.34 146.05 0) (fields_autoplaced)
+    (effects (font (size 1.27 1.27)) (justify left bottom))
+  )
+  (label "LHLED" (at 180.34 139.7 0) (fields_autoplaced)
+    (effects (font (size 1.27 1.27)) (justify left bottom))
+  )
   (label "SCHLUSS-" (at 119.38 196.85 0) (fields_autoplaced)
     (effects (font (size 1.27 1.27)) (justify left bottom))
@@
   )
   (label "LV" (at 180.34 81.28 0) (fields_autoplaced)
+    (effects (font (size 1.27 1.27)) (justify left bottom))
+  )
+  (label "BRIDGE+" (at 175.26 50.8 0) (fields_autoplaced)
     (effects (font (size 1.27 1.27)) (justify left bottom))
   )
@@
     )
   )
-  (symbol (lib_id "Jumper:SolderJumper_2_Open") (at 142.24 33.02 0) (unit 1)
-    (in_bom yes) (on_board yes) (dnp no) (fields_autoplaced)
-    (property "Reference" "JP1" (at 142.24 29.1211 0)
-      (effects (font (size 1.27 1.27)))
-    )
-    (property "Value" "SolderJumper_2_Open" (at 142.24 31.0421 0)
-      (effects (font (size 1.27 1.27)))
-    )
-    (property "Footprint" "Jumper:SolderJumper-2_P1.3mm_Open_RoundedPad1.0x1.5mm" (at 142.24 33.02 0)
-      (effects (font (size 1.27 1.27)) hide)
-    )
-    (property "Datasheet" "~" (at 142.24 33.02 0)
+  (symbol (lib_id "Jumper:SolderJumper_2_Open") (at 133.35 43.18 90) (unit 1)
+    (in_bom yes) (on_board yes) (dnp no)
+    (property "Reference" "JP1" (at 135.89 41.91 90)
+      (effects (font (size 1.27 1.27)) (justify right))
+    )
+    (property "Value" "SolderJumper_2_Open" (at 135.89 44.45 90)
+      (effects (font (size 1.27 1.27)) (justify right))
+    )
+    (property "Footprint" "Jumper:SolderJumper-2_P1.3mm_Open_RoundedPad1.0x1.5mm" (at 133.35 43.18 0)
+      (effects (font (size 1.27 1.27)) hide)
+    )
+    (property "Datasheet" "~" (at 133.35 43.18 0)
       (effects (font (size 1.27 1.27)) hide)
     )
@@
       (effects (font (size 1.27 1.27)) (justify left))
     )
-    (property "Footprint" "TestPoint:TestPoint_Pad_1.5x1.5mm" (at 267.97 45.72 0)
+    (property "Footprint" "Local:Minitrix_Pad" (at 267.97 45.72 0)
       (effects (font (size 1.27 1.27)) hide)
     )
@@
     )
   )
-  (symbol (lib_id "Jumper:SolderJumper_2_Open") (at 175.26 33.02 0) (unit 1)
+  (symbol (lib_id "Jumper:SolderJumper_2_Open") (at 166.37 43.18 90) (unit 1)
     (in_bom yes) (on_board yes) (dnp no)
-    (property "Reference" "JP2" (at 175.26 29.1211 0)
-      (effects (font (size 1.27 1.27)))
-    )
-    (property "Value" "SolderJumper_2_Open" (at 175.26 31.0421 0)
-      (effects (font (size 1.27 1.27)))
-    )
-    (property "Footprint" "Jumper:SolderJumper-2_P1.3mm_Open_RoundedPad1.0x1.5mm" (at 175.26 33.02 0)
-      (effects (font (size 1.27 1.27)) hide)
-    )
-    (property "Datasheet" "~" (at 175.26 33.02 0)
+    (property "Reference" "JP2" (at 170.18 41.91 90)
+      (effects (font (size 1.27 1.27)) (justify right))
+    )
+    (property "Value" "SolderJumper_2_Open" (at 170.18 44.45 90)
+      (effects (font (size 1.27 1.27)) (justify right))
+    )
+    (property "Footprint" "Jumper:SolderJumper-2_P1.3mm_Open_RoundedPad1.0x1.5mm" (at 166.37 43.18 0)
+      (effects (font (size 1.27 1.27)) hide)
+    )
+    (property "Datasheet" "~" (at 166.37 43.18 0)
       (effects (font (size 1.27 1.27)) hide)
     )
@@
       (effects (font (size 1.27 1.27)) (justify left))
     )
-    (property "Footprint" "TestPoint:TestPoint_Pad_1.5x1.5mm" (at 267.97 21.59 0)
-      (effects (font (size 1.27 1.27)) hide)
-    )
+    (property "Footprint" "Local:Minitrix_Pad" (at 267.97 21.59 0)
+      (effects (font (size 1.27 1.27)) hide)
+    )
